File: PDB v1.4/source/PDB1.4/PDB1.4.kicad_pcb (KiCad board)
At the start: 6 copper layers, 86.5 x 150 mm, 38 parts, among them J1 TFM-107-02-L-D-WT, J10 2132250430, J2 1719710105, J3 1719710105, J4 1719710105, J5 1719710105, J6 2132250430, J7 1719710106, J8 2132250430, J9 2132250430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

Commit message: Add board Name
Other:
- board text added: "PDB v1.4"
Changed lines of the file:
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@@
 			(drillshape 0)
 			(scaleselection 1)
-			(outputdirectory "../../production/gerber/")
+			(outputdirectory "../../production/JLCPCB/gerber/")
 		)
 	)
@@
 		(at 85.063374 149.059263 -98)
 		(property "Reference" "J2"
-			(at 3.638962 -1.41686 -98)
+			(at 4.181415 -3.017937 82)
 			(layer "F.SilkS")
-			(hide yes)
 			(effects
 				(font
-					(size 1 1)
-					(thickness 0.15)
+					(size 1.5 1.5)
+					(thickness 0.2)
 				)
 			)
 		)
 		(property "Value" "1719710105"
-			(at -7.9 3.65 -98)
+			(at -7.9 3.65 82)
 			(layer "F.Fab")
 			(effects
@@
 		)
 		(fp_text user "PTH D1.09 +/- 0.08"
-			(at -12.740001 6.6724 -98)
+			(at -12.740001 6.6724 82)
 			(layer "F.Fab")
 			(effects
@@
 		(at 130.88 144.13)
 		(property "Reference" "J8"
-			(at 6.53 2.32 0)
+			(at 7.56 -2.48 0)
 			(layer "F.SilkS")
-			(hide yes)
 			(effects
 				(font
-					(size 1 1)
-					(thickness 0.15)
+					(size 1.5 1.5)
+					(thickness 0.2)
 				)
 			)
@@
 			(at 3.76 7.045 0)
 			(layer "F.Fab")
+			(hide yes)
 			(effects
 				(font
@@
 			(unlocked yes)
 			(layer "B.SilkS")
+			(hide yes)
 			(effects
 				(font
@@
 			(unlocked yes)
 			(layer "B.SilkS")
+			(hide yes)
 			(effects
 				(font
@@
 			(unlocked yes)
 			(layer "B.SilkS")
+			(hide yes)
 			(effects
 				(font
@@
 		(at 162.340653 139.224363 98)
 		(property "Reference" "J3"
-			(at -11.574477 -5.096455 -82)
+			(at -11.594571 -5.417023 98)
 			(layer "F.SilkS")
-			(hide yes)
 			(effects
 				(font
-					(size 1 1)
-					(thickness 0.15)
+					(size 1.5 1.5)
+					(thickness 0.2)
 				)
 			)
@@
 		(at 101 144)
 		(property "Reference" "J6"
-			(at 4.3 3.6 0)
+			(at 7.55 -2.4 0)
 			(layer "F.SilkS")
-			(hide yes)
 			(effects
 				(font
-					(size 1 1)
-					(thickness 0.15)
+					(size 1.5 1.5)
+					(thickness 0.2)
 				)
 			)
@@
 			(at 3.76 7.045 0)
 			(layer "F.Fab")
+			(hide yes)
 			(effects
 				(font
@@
 		(at 147.88 144.13 180)
 		(property "Reference" "J9"
-			(at -2.475 5.79 0)
+			(at 7.46 2.55 0)
 			(layer "B.SilkS")
-			(hide yes)
 			(effects
 				(font
-					(size 1 1)
-					(thickness 0.15)
+					(size 1.5 1.5)
+					(thickness 0.2)
 				)
 				(justify mirror)
@@
 		(at 158.188059 146.788397 98)
 		(property "Reference" "J1"
-			(at -4.859999 4.384999 98)
+			(at -6.076964 -4.194631 -82)
 			(layer "B.SilkS")
-			(hide yes)
 			(effects
 				(font
-					(size 1 1)
-					(thickness 0.15)
+					(size 1.5 1.5)
+					(thickness 0.2)
 				)
 				(justify mirror)
@@
 		(at 92.347741 140.944663 83)
 		(property "Reference" "J7"
-			(at 2.122866 14.311329 -7)
+			(at -14.193809 5.311641 83)
 			(layer "B.SilkS")
-			(hide yes)
 			(effects
 				(font
-					(size 1 1)
-					(thickness 0.15)
+					(size 1.5 1.5)
+					(thickness 0.2)
 				)
 				(justify mirror)
@@
 		(at 89.229347 123.884363 82)
 		(property "Reference" "J4"
-			(at -11.829398 4.823933 -98)
+			(at 1.343148 5.21447 -98)
 			(layer "B.SilkS")
-			(hide yes)
 			(effects
 				(font
-					(size 1 1)
-					(thickness 0.15)
+					(size 1.5 1.5)
+					(thickness 0.2)
 				)
 				(justify mirror)
@@
 		(at 117.89 144.28 180)
 		(property "Reference" "J10"
-			(at -4.8 -4.49 0)
+			(at 8.14 2.53 0)
 			(layer "B.SilkS")
-			(hide yes)
 			(effects
 				(font
-					(size 1 1)
-					(thickness 0.15)
+					(size 1.5 1.5)
+					(thickness 0.2)
 				)
 				(justify mirror)
@@
 		(at 161.102372 133.977389 -82)
 		(property "Reference" "J5"
-			(at 1.716435 5.050404 -82)
+			(at -11.28204 5.495699 98)
 			(layer "B.SilkS")
-			(hide yes)
 			(effects
 				(font
-					(size 1 1)
-					(thickness 0.15)
+					(size 1.5 1.5)
+					(thickness 0.2)
 				)
 				(justify mirror)
@@
 		)
 		(property "Value" "1719710105"
-			(at -2.53 -5.043 -82)
+			(at -2.53 -5.043 98)
 			(layer "B.Fab")
 			(effects
@@
 		)
 		(fp_text user "PTH D1.09 +/- 0.08"
-			(at -12.74 -6.6724 -82)
+			(at -12.74 -6.6724 98)
 			(layer "B.Fab")
 			(effects
@@
 		(layer "B.Mask")
 	)
-	(gr_line
-		(start 150.526998 156.650042)
-		(end 98.595273 156.651928)
-		(stroke
-			(width 1)
-			(type default)
-		)
-		(layer "B.Mask")
-	)
 	(gr_arc
 		(start 162.103521 159.01)
@@
 	)
 	(gr_arc
-		(start 96.883521 157.62)
-		(mid 97.612197 156.911047)
-		(end 98.595273 156.651928)
-		(stroke
-			(width 1)
-			(type default)
-		)
-		(layer "B.Mask")
-	)
-	(gr_arc
 		(start 85.553521 155.72)
 		(mid 82.665358 152.032725)
@@
 		(layer "B.Mask")
 	)
-	(gr_arc
-		(start 150.526998 156.650042)
-		(mid 151.521691 156.914875)
-		(end 152.252908 157.639356)
-		(stroke
-			(width 1)
-			(type default)
-		)
-		(layer "B.Mask")
-	)
 	(gr_line
 		(start 91.77 165.24)
@@
 		(layer "Edge.Cuts")
 	)
+	(gr_text "PDB v1.4"
+		(at 117 37.91 0)
+		(layer "F.Cu")
+		(effects
+			(font
+				(size 2 2)
+				(thickness 0.3)
+				(bold yes)
+			)
+			(justify left bottom)
+		)
+	)
 	(segment
